Commit message: integrated world with arena

File: rover_description/urdf/rover.xacro (robot description, xacro)
@@ -238,3 +238,18 @@
     <self_collide>1</self_collide>
   </gazebo>
+  <gazebo reference="upper_plate">
+    <material>Gazebo/Orange</material>
+  </gazebo>
+    <gazebo reference="liwheel_rightnk1">
+    <material>Gazebo/Orange</material>
+  </gazebo>
+    <gazebo reference="wheel_right">
+    <material>Gazebo/Orange</material>
+  </gazebo>
+  <gazebo reference="wheel_left">
+    <material>Gazebo/Orange</material>
+  </gazebo>
+    <gazebo reference="base_link">
+    <material>Gazebo/White</material>
+  </gazebo>
 </robot>
