Commit message: 3rd party packages added, Main packages combined

File: rover_description/urdf/birds_eye_cam.xacro (robot description, xacro)
@@ -1,4 +1,4 @@
 <?xml version="1.0"?>
-<robot name="aRm" xmlns:xacro="http://ros.org/wiki/xacro">
+<robot name="cam_bot" xmlns:xacro="http://ros.org/wiki/xacro">
 <!-- <link name="world" />
 <joint name="world_base" type="fixed">
@@ -8,9 +8,30 @@
 </joint> -->
 <link name="base_link">
+<inertial>
+        <mass value="1.584994"/>
+        <origin xyz="0.0 0.0 0.0"/>
+        <inertia
+          ixx="0.01042" ixy="0.001177" ixz="-0.0008871"
+          iyy="0.01045" iyz="0.0002226"
+          izz="0.01817"/>
+      </inertial>
+    <visual>
+        <geometry>
+          <mesh filename="package://rover_description/meshes/dae_markers/test_modified.dae"/>
+        </geometry>
+        <!-- <material name="RED"> -->
+          <!-- <color rgba="1.0 0.0 0.0 1.0"/> -->
+        <!-- </material> -->
+      </visual>
+      <collision>
+        <geometry>
+          <mesh filename="package://rover_description/meshes/dae_markers/test_modified.dae" />
+        </geometry>
+      </collision>
 </link>
 <joint name="camera_to_base" type="fixed">
       <parent link="base_link" />
       <child link = "camera_link" />
-      <origin xyz="0.0 0.0 3.0" rpy="0.0 0.0 0.0" />
+      <origin xyz="0.0 0.0 3.0" rpy="3.142 0.0 0.0" />
       <axis xyz="0 0 1" />
       <limit lower="-3.142" upper="3.142" effort="150.0" velocity="1.5"/>

Commit message: arena texture added

File: rover_description/urdf/birds_eye_cam.xacro (robot description, xacro)
@@ -18,5 +18,5 @@
     <visual>
         <geometry>
-          <mesh filename="package://rover_description/meshes/dae_markers/test_modified.dae"/>
+          <mesh filename="package://rover_sim/arena/arena/arena_one.dae"/>
         </geometry>
         <!-- <material name="RED"> -->
@@ -26,5 +26,5 @@
       <collision>
         <geometry>
-          <mesh filename="package://rover_description/meshes/dae_markers/test_modified.dae" />
+          <mesh filename="package://rover_sim/arena/arena/arena_one.dae" />
         </geometry>
       </collision>

Commit message: stable version achieved

File: rover_description/urdf/birds_eye_cam.xacro (robot description, xacro)
@@ -1,11 +1,11 @@
 <?xml version="1.0"?>
 <robot name="cam_bot" xmlns:xacro="http://ros.org/wiki/xacro">
-<!-- <link name="world" />
+<link name="world" />
 <joint name="world_base" type="fixed">
     <parent link="world" />
-    <child link="base_link"/>
-    <origin xyz="0.0 0.0 0.0" rpy="0.0 0.0 0.0" />
-</joint> -->
-<link name="base_link">
+    <child link="camera_base_link"/>
+    <origin xyz="-0.4 0.0 0.0" rpy="0.0 0.0 0.0" />
+</joint>
+<link name="camera_base_link">
 <inertial>
         <mass value="1.584994"/>
@@ -18,5 +18,5 @@
     <visual>
         <geometry>
-          <mesh filename="package://rover_sim/arena/arena/arena_one.dae"/>
+          <box size="0.001 0.001 0.001" />
         </geometry>
         <!-- <material name="RED"> -->
@@ -26,16 +26,73 @@
       <collision>
         <geometry>
-          <mesh filename="package://rover_sim/arena/arena/arena_one.dae" />
+          <box size="0.001 0.001 0.001" />
         </geometry>
       </collision>
 </link>
 <joint name="camera_to_base" type="fixed">
-      <parent link="base_link" />
+      <parent link="camera_base_link" />
       <child link = "camera_link" />
-      <origin xyz="0.0 0.0 3.0" rpy="3.142 0.0 0.0" />
+      <origin xyz="0.0 0.0 2.0" rpy="0 1.57 0.0" />
       <axis xyz="0 0 1" />
       <limit lower="-3.142" upper="3.142" effort="150.0" velocity="1.5"/>
 </joint>
 <link name="camera_link">
+<inertial>
+        <mass value="1.584994"/>
+        <origin xyz="0.0 0.0 0.0"/>
+        <inertia
+          ixx="0.01042" ixy="0.001177" ixz="-0.0008871"
+          iyy="0.01045" iyz="0.0002226"
+          izz="0.01817"/>
+      </inertial>
+    <visual>
+        <geometry>
+        <box size="0.001 0.001 0.001" />
+        </geometry>
+      </visual>
+      <collision>
+        <geometry>
+        <box size="0.001 0.001 0.001" />
+        </geometry>
+      </collision>
 </link>
+<gazebo reference="camera_link">
+    <sensor type="camera" name="camera">
+      <update_rate>30.0</update_rate>
+      <camera name="head">
+        <horizontal_fov>1.3962634</horizontal_fov>
+        <image>
+          <width>640</width>
+          <height>480</height>
+          <format>R8G8B8</format>
+        </image>
+        <clip>
+          <near>0.02</near>
+          <far>300</far>
+        </clip>
+        <noise>
+          <type>gaussian</type>
+          <!-- Noise is sampled independently per pixel on each frame.
+               That pixel's noise value is added to each of its color
+               channels, which at that point lie in the range [0,1]. -->
+          <mean>0.0</mean>
+          <stddev>0.007</stddev>
+        </noise>
+      </camera>
+      <plugin name="camera_controller" filename="libgazebo_ros_camera.so">
+        <alwaysOn>true</alwaysOn>
+        <updateRate>0.0</updateRate>
+        <cameraName>usb_cam</cameraName>
+        <imageTopicName>image_raw</imageTopicName>
+        <cameraInfoTopicName>/camera/camera_info</cameraInfoTopicName>
+        <frameName>camera_link</frameName>
+        <hackBaseline>0.07</hackBaseline>
+        <distortionK1>0.0</distortionK1>
+        <distortionK2>0.0</distortionK2>
+        <distortionK3>0.0</distortionK3>
+        <distortionT1>0.0</distortionT1>
+        <distortionT2>0.0</distortionT2>
+      </plugin>
+    </sensor>
+  </gazebo>
 </robot>

Commit message: Aruco tags generated

File: rover_description/urdf/birds_eye_cam.xacro (robot description, xacro)
@@ -5,5 +5,5 @@
     <parent link="world" />
     <child link="camera_base_link"/>
-    <origin xyz="-0.4 0.0 0.0" rpy="0.0 0.0 0.0" />
+    <origin xyz="0 0.0 0.0" rpy="0.0 0.0 0.0" />
 </joint>
 <link name="camera_base_link">
@@ -33,7 +33,5 @@
       <parent link="camera_base_link" />
       <child link = "camera_link" />
-      <origin xyz="0.0 0.0 2.0" rpy="0 1.57 0.0" />
-      <axis xyz="0 0 1" />
-      <limit lower="-3.142" upper="3.142" effort="150.0" velocity="1.5"/>
+      <origin xyz="0.0 0.0 2" rpy="0 3.142 0.0" />
 </joint>
 <link name="camera_link">
